Commit message: FIXED (hopefully)
URDF file has a base link. Also, defined gravity in compensation code.

File: src/arm.urdf (robot description, URDF)
Before this commit: robot two_dof_arm, 2 links, 2 joints
Links:
- added link world
Joints:
- joint joint1: axis 1 0 0 -> 0 0 1; limit (none) -> lower=-1.57 upper=1.57 effort=11 velocity=20; parent base_link -> world
- joint joint2: axis 1 0 0 -> 0 0 1; limit (none) -> lower=-1.57 upper=1.57 effort=11 velocity=20; origin xyz=0.310 0 0 rpy=0 0 0 -> xyz=0.45 0 0 rpy=0 0 0

Commit message: Changed URDF + prep for testing

File: src/arm.urdf (robot description, URDF)
Before this commit: robot two_dof_arm, 3 links, 2 joints
Links:
- link link1: geometry visual cylinder length=0.32 radius=0.05
- link link2: geometry visual cylinder length=0.26 radius=0.05
- link world: geometry visual box size=0.1 0.1 0.1
Joints:
- joint joint1: axis 0 0 1 -> 0 1 0; limit lower=-1.57 upper=1.57 effort=11 velocity=20 -> lower=-1.57 upper=1.57 effort=8 velocity=20
- joint joint2: axis 0 0 1 -> 0 1 0; limit lower=-1.57 upper=1.57 effort=11 velocity=20 -> lower=-1.57 upper=1.57 effort=8 velocity=20; origin xyz=0.45 0 0 rpy=0 0 0 -> xyz=0 0 -0.32 rpy=0 0 0
